File: USB.kicad_blocks/UBS-type-C_31-M-12.kicad_block/UBS-type-C_31-M-12.kicad_sch (KiCad schematic)
At the start: 4 parts, among them J1 USB_C_Receptacle_USB2.0_16P, U1 USBLC6-2SC6

Commit message: USBc upgrade
Parts:
- J1: LCSC (none) -> C165948
- U1: LCSC (none) -> C2827654
