File: src/UBS-C_TYPE-C-31-M-12/UBS-C_TYPE-C-31-M-12.kicad_sch (KiCad schematic)
At the start: 4 parts, among them J1 USB_C_Receptacle_USB2.0_16P, U1 USBLC6-2SC6

Commit message: USBc upgrade
Parts:
- J1: LCSC (none) -> C165948
- U1: LCSC (none) -> C2827654
Changed lines of the file:
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@@
+			)
+		)
+		(property "LCSC" "C2827654"
+			(at 160.02 82.55 0)
+			(hide yes)
+			(show_name no)
+			(do_not_autoplace no)
+			(effects
+				(font
+					(size 1.27 1.27)
+				)
 			)
 		)
@@
 			(at 118.11 82.55 0)
 			(hide yes)
+			(show_name no)
+			(do_not_autoplace no)
+			(effects
+				(font
+					(size 1.27 1.27)
+				)
+			)
+		)
+		(property "LCSC" "C165948"
+			(at 118.11 82.55 0)
+			(hide yes)

Commit message: forgor to version
Other:
- title: (none) -> USB C design block
Changed lines of the file:
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@@
 	(generator_version "10.0")
 	(paper "A4")
+	(title_block
+		(title "USB C design block")
+		(rev "V1")
+	)
 	(text "500mA - 3A @ 5V"
 		(exclude_from_sim no)
